File: pcb/EduRov-motherboard/MotorController.sch (KiCad schematic (older format))
At the start: 10 parts, among them IC201 L6203, U201 ACS723xLCTR-05AB

Commit message: Update PCBs after prototyping
Parts:
- removed IC201: L6203, EduROV:MULTIWATT-11, symbol eduROV_motherboard:L6203
- added IC401: L6203, SnapEDA Library:MULTIWATT-11, symbol L6203:L6203
Changed lines of the file:
@@
 $Descr A4 11693 8268
 encoding utf-8
-Sheet 2 5
+Sheet 4 5
 Title ""
 Date ""
@@
 AR Path="/6003F027/5FFEEEFF" Ref="D402"  Part="1"
 AR Path="/60043462/5FFEEEFF" Ref="D502"  Part="1"
-F 0 "D502" H 6450 3500 50  0000 C CNN
+F 0 "D402" H 6450 3500 50  0000 C CNN
 F 1 "D" H 6400 3400 50  0001 C CNN
 F 2 "Diode_THT:D_DO-41_SOD81_P3.81mm_Vertical_KathodeUp" H 6250 3450 50  0001 C CNN
@@
 AR Path="/6003F027/5FFEEF0B" Ref="D401"  Part="1"
 AR Path="/60043462/5FFEEF0B" Ref="D501"  Part="1"
-F 0 "D501" H 6300 3500 50  0000 C CNN
+F 0 "D401" H 6300 3500 50  0000 C CNN
 F 1 "D" H 6250 3400 50  0001 C CNN
 F 2 "Diode_THT:D_DO-41_SOD81_P3.81mm_Vertical_KathodeUp" H 6100 3450 50  0001 C CNN
@@
 Wire Wire Line
 	2900 3000 4200 3000
-$Comp
-L eduROV_motherboard:L6203 IC?
-U 1 1 5FFEEF31
-P 4800 3100
-AR Path="/5FFEEF31" Ref="IC?"  Part="1"
-AR Path="/5FFEC45F/5FFEEF31" Ref="IC201"  Part="1"
-AR Path="/60017CE1/5FFEEF31" Ref="IC?"  Part="1"
-AR Path="/600184A3/5FFEEF31" Ref="IC?"  Part="1"
-AR Path="/60018874/5FFEEF31" Ref="IC?"  Part="1"
-AR Path="/6003A868/5FFEEF31" Ref="IC301"  Part="1"
-AR Path="/6003F027/5FFEEF31" Ref="IC401"  Part="1"
-AR Path="/60043462/5FFEEF31" Ref="IC501"  Part="1"
-F 0 "IC501" H 4400 3550 50  0000 C CNN
-F 1 "L6203" H 4400 3450 50  0000 C CNN
-F 2 "EduROV:MULTIWATT-11" H 4800 3100 50  0001 L BNN
-F 3 "" H 4800 3100 50  0001 L BNN
-F 4 "" H 4800 3100 50  0001 L BNN "MF"
-F 5 "56P8434" H 4800 3100 50  0001 L BNN "OC_NEWARK"
-F 6 "1467715" H 4800 3100 50  0001 L BNN "OC_FARNELL"
-F 7 "L6203" H 4800 3100 50  0001 L BNN "MPN"
-	1    4800 3100
-	1    0    0    -1
-$EndComp
 Text GLabel 6250 3750 3    60   Input ~ 0
 GND
@@
 AR Path="/6003F027/5FFEEF49" Ref="C404"  Part="1"
 AR Path="/60043462/5FFEEF49" Ref="C504"  Part="1"
-F 0 "C504" V 5600 2850 50  0000 C CNN
+F 0 "C404" V 5600 2850 50  0000 C CNN
 F 1 "15nF" V 5600 3150 50  0000 C CNN
 F 2 "Capacitor_THT:C_Disc_D3.8mm_W2.6mm_P2.50mm" H 5650 3000 50  0001 C CNN
@@
 AR Path="/6003F027/5FFEEF54" Ref="C405"  Part="1"
 AR Path="/60043462/5FFEEF54" Ref="C505"  Part="1"
-F 0 "C505" V 5700 3150 50  0000 C CNN
+F 0 "C405" V 5700 3150 50  0000 C CNN
 F 1 "15nF" V 5700 3450 50  0000 C CNN
 F 2 "Capacitor_THT:C_Disc_D3.8mm_W2.6mm_P2.50mm" H 5650 3300 50  0001 C CNN
@@
 AR Path="/6003F027/5FFEEF6B" Ref="C402"  Part="1"
 AR Path="/60043462/5FFEEF6B" Ref="C502"  Part="1"
-F 0 "C502" V 3850 2750 50  0000 C CNN
+F 0 "C402" V 3850 2750 50  0000 C CNN
 F 1 "220nF" V 3850 3050 50  0000 C CNN
 F 2 "Capacitor_THT:C_Disc_D3.8mm_W2.6mm_P2.50mm" H 3900 2900 50  0001 C CNN
@@
 AR Path="/6003A868/600F7A3C" Ref="C303"  Part="1"
 AR Path="/6003F027/600F7A3C" Ref="C403"  Part="1"
-F 0 "C503" V 5300 2650 50  0000 C CNN
+F 0 "C403" V 5300 2650 50  0000 C CNN
 F 1 "100nF" V 5200 2700 50  0000 C CNN
 F 2 "Capacitor_THT:C_Disc_D5.0mm_W2.5mm_P2.50mm" H 5188 2350 50  0001 C CNN
@@
 AR Path="/6003F027/6032BA93" Ref="R401"  Part="1"
 AR Path="/60043462/6032BA93" Ref="R501"  Part="1"
-F 0 "R501" V 3880 4200 50  0000 C CNN
+F 0 "R401" V 3880 4200 50  0000 C CNN
 F 1 "0" V 3800 4200 50  0000 C CNN
 F 2 "Resistor_THT:R_Axial_DIN0204_L3.6mm_D1.6mm_P1.90mm_Vertical" V 3730 4200 50  0001 C CNN
@@
 AR Path="/6003F027/60485F83" Ref="U401"  Part="1"
 AR Path="/60043462/60485F83" Ref="U501"  Part="1"
-F 0 "U501" H 3000 4700 50  0000 C CNN
+F 0 "U401" H 3000 4700 50  0000 C CNN
 F 1 "ACS723xLCTR-05AB" H 3250 4600 50  0000 C CNN
 F 2 "Package_SO:SOIC-8_3.9x4.9mm_P1.27mm" H 2850 3900 50  0001 L CIN
@@
 AR Path="/6003A868/60487676" Ref="C301"  Part="1"
 AR Path="/6003F027/60487676" Ref="C401"  Part="1"
-F 0 "C501" V 3100 3950 50  0000 C CNN
+F 0 "C401" V 3100 3950 50  0000 C CNN
 F 1 "100nF" V 3000 4000 50  0000 C CNN
 F 2 "Capacitor_THT:C_Disc_D5.0mm_W2.5mm_P2.50mm" H 2938 3650 50  0001 C CNN
@@
 Wire Notes Line
 	3650 5100 3650 3400
+$Comp
+L L6203:L6203 IC401
+U 1 1 60738BFF
+P 4800 3100
+AR Path="/6003F027/60738BFF" Ref="IC401"  Part="1"
+AR Path="/5FFEC45F/60738BFF" Ref="IC201"  Part="1"
+AR Path="/6003A868/60738BFF" Ref="IC301"  Part="1"
+AR Path="/60043462/60738BFF" Ref="IC501"  Part="1"
+F 0 "IC401" H 4800 3681 50  0000 C CNN
+F 1 "L6203" H 4800 3590 50  0000 C CNN
+F 2 "SnapEDA Library:MULTIWATT-11" H 4800 3100 50  0001 L BNN
+F 3 "" H 4800 3100 50  0001 L BNN
+F 4 "" H 4800 3100 50  0001 L BNN "MF"
+F 5 "56P8434" H 4800 3100 50  0001 L BNN "OC_NEWARK"
+F 6 "1467715" H 4800 3100 50  0001 L BNN "OC_FARNELL"
+F 7 "L6203" H 4800 3100 50  0001 L BNN "MPN"
+	1    4800 3100
+	1    0    0    -1
+$EndComp
 $EndSCHEMATC

Commit message: Update schematic.
Changed lines of the file:
@@
 AR Path="/6003F027/5FFEEEFF" Ref="D402"  Part="1"
 AR Path="/60043462/5FFEEEFF" Ref="D502"  Part="1"
-F 0 "D402" H 6450 3500 50  0000 C CNN
+F 0 "D502" H 6450 3500 50  0000 C CNN
 F 1 "D" H 6400 3400 50  0001 C CNN
 F 2 "Diode_THT:D_DO-41_SOD81_P3.81mm_Vertical_KathodeUp" H 6250 3450 50  0001 C CNN
@@
 AR Path="/6003F027/5FFEEF0B" Ref="D401"  Part="1"
 AR Path="/60043462/5FFEEF0B" Ref="D501"  Part="1"
-F 0 "D401" H 6300 3500 50  0000 C CNN
+F 0 "D501" H 6300 3500 50  0000 C CNN
 F 1 "D" H 6250 3400 50  0001 C CNN
 F 2 "Diode_THT:D_DO-41_SOD81_P3.81mm_Vertical_KathodeUp" H 6100 3450 50  0001 C CNN
@@
 AR Path="/6003F027/5FFEEF49" Ref="C404"  Part="1"
 AR Path="/60043462/5FFEEF49" Ref="C504"  Part="1"
-F 0 "C404" V 5600 2850 50  0000 C CNN
+F 0 "C504" V 5600 2850 50  0000 C CNN
 F 1 "15nF" V 5600 3150 50  0000 C CNN
 F 2 "Capacitor_THT:C_Disc_D3.8mm_W2.6mm_P2.50mm" H 5650 3000 50  0001 C CNN
@@
 AR Path="/6003F027/5FFEEF54" Ref="C405"  Part="1"
 AR Path="/60043462/5FFEEF54" Ref="C505"  Part="1"
-F 0 "C405" V 5700 3150 50  0000 C CNN
+F 0 "C505" V 5700 3150 50  0000 C CNN
 F 1 "15nF" V 5700 3450 50  0000 C CNN
 F 2 "Capacitor_THT:C_Disc_D3.8mm_W2.6mm_P2.50mm" H 5650 3300 50  0001 C CNN
@@
 AR Path="/6003F027/5FFEEF6B" Ref="C402"  Part="1"
 AR Path="/60043462/5FFEEF6B" Ref="C502"  Part="1"
-F 0 "C402" V 3850 2750 50  0000 C CNN
+F 0 "C502" V 3850 2750 50  0000 C CNN
 F 1 "220nF" V 3850 3050 50  0000 C CNN
 F 2 "Capacitor_THT:C_Disc_D3.8mm_W2.6mm_P2.50mm" H 3900 2900 50  0001 C CNN
@@
 AR Path="/6003A868/600F7A3C" Ref="C303"  Part="1"
 AR Path="/6003F027/600F7A3C" Ref="C403"  Part="1"
-F 0 "C403" V 5300 2650 50  0000 C CNN
+F 0 "C503" V 5300 2650 50  0000 C CNN
 F 1 "100nF" V 5200 2700 50  0000 C CNN
 F 2 "Capacitor_THT:C_Disc_D5.0mm_W2.5mm_P2.50mm" H 5188 2350 50  0001 C CNN
@@
 AR Path="/6003F027/6032BA93" Ref="R401"  Part="1"
 AR Path="/60043462/6032BA93" Ref="R501"  Part="1"
-F 0 "R401" V 3880 4200 50  0000 C CNN
+F 0 "R501" V 3880 4200 50  0000 C CNN
 F 1 "0" V 3800 4200 50  0000 C CNN
 F 2 "Resistor_THT:R_Axial_DIN0204_L3.6mm_D1.6mm_P1.90mm_Vertical" V 3730 4200 50  0001 C CNN
@@
 AR Path="/6003F027/60485F83" Ref="U401"  Part="1"
 AR Path="/60043462/60485F83" Ref="U501"  Part="1"
-F 0 "U401" H 3000 4700 50  0000 C CNN
+F 0 "U501" H 3000 4700 50  0000 C CNN
 F 1 "ACS723xLCTR-05AB" H 3250 4600 50  0000 C CNN
 F 2 "Package_SO:SOIC-8_3.9x4.9mm_P1.27mm" H 2850 3900 50  0001 L CIN
@@
 AR Path="/6003A868/60487676" Ref="C301"  Part="1"
 AR Path="/6003F027/60487676" Ref="C401"  Part="1"
-F 0 "C401" V 3100 3950 50  0000 C CNN
+F 0 "C501" V 3100 3950 50  0000 C CNN
 F 1 "100nF" V 3000 4000 50  0000 C CNN
 F 2 "Capacitor_THT:C_Disc_D5.0mm_W2.5mm_P2.50mm" H 2938 3650 50  0001 C CNN
@@
 AR Path="/6003A868/60738BFF" Ref="IC301"  Part="1"
 AR Path="/60043462/60738BFF" Ref="IC501"  Part="1"
-F 0 "IC401" H 4800 3681 50  0000 C CNN
+F 0 "IC501" H 4800 3681 50  0000 C CNN
 F 1 "L6203" H 4800 3590 50  0000 C CNN
 F 2 "SnapEDA Library:MULTIWATT-11" H 4800 3100 50  0001 L BNN

Commit message: Add L6203 to edurov library
Parts:
- IC401: symbol L6203:L6203 -> Edurov:L6203
Changed lines of the file:
@@
 $Descr A4 11693 8268
 encoding utf-8
-Sheet 4 5
+Sheet 2 5
 Title ""
 Date ""
@@
 AR Path="/6003F027/5FFEEEFF" Ref="D402"  Part="1"
 AR Path="/60043462/5FFEEEFF" Ref="D502"  Part="1"
-F 0 "D502" H 6450 3500 50  0000 C CNN
+F 0 "D202" H 6450 3500 50  0000 C CNN
 F 1 "D" H 6400 3400 50  0001 C CNN
 F 2 "Diode_THT:D_DO-41_SOD81_P3.81mm_Vertical_KathodeUp" H 6250 3450 50  0001 C CNN
@@
 AR Path="/6003F027/5FFEEF0B" Ref="D401"  Part="1"
 AR Path="/60043462/5FFEEF0B" Ref="D501"  Part="1"
-F 0 "D501" H 6300 3500 50  0000 C CNN
+F 0 "D201" H 6300 3500 50  0000 C CNN
 F 1 "D" H 6250 3400 50  0001 C CNN
 F 2 "Diode_THT:D_DO-41_SOD81_P3.81mm_Vertical_KathodeUp" H 6100 3450 50  0001 C CNN
@@
 AR Path="/6003F027/5FFEEF49" Ref="C404"  Part="1"
 AR Path="/60043462/5FFEEF49" Ref="C504"  Part="1"
-F 0 "C504" V 5600 2850 50  0000 C CNN
+F 0 "C204" V 5600 2850 50  0000 C CNN
 F 1 "15nF" V 5600 3150 50  0000 C CNN
 F 2 "Capacitor_THT:C_Disc_D3.8mm_W2.6mm_P2.50mm" H 5650 3000 50  0001 C CNN
@@
 AR Path="/6003F027/5FFEEF54" Ref="C405"  Part="1"
 AR Path="/60043462/5FFEEF54" Ref="C505"  Part="1"
-F 0 "C505" V 5700 3150 50  0000 C CNN
+F 0 "C205" V 5700 3150 50  0000 C CNN
 F 1 "15nF" V 5700 3450 50  0000 C CNN
 F 2 "Capacitor_THT:C_Disc_D3.8mm_W2.6mm_P2.50mm" H 5650 3300 50  0001 C CNN
@@
 AR Path="/6003F027/5FFEEF6B" Ref="C402"  Part="1"
 AR Path="/60043462/5FFEEF6B" Ref="C502"  Part="1"
-F 0 "C502" V 3850 2750 50  0000 C CNN
+F 0 "C202" V 3850 2750 50  0000 C CNN
 F 1 "220nF" V 3850 3050 50  0000 C CNN
 F 2 "Capacitor_THT:C_Disc_D3.8mm_W2.6mm_P2.50mm" H 3900 2900 50  0001 C CNN
@@
 AR Path="/6003A868/600F7A3C" Ref="C303"  Part="1"
 AR Path="/6003F027/600F7A3C" Ref="C403"  Part="1"
-F 0 "C503" V 5300 2650 50  0000 C CNN
+F 0 "C203" V 5300 2650 50  0000 C CNN
 F 1 "100nF" V 5200 2700 50  0000 C CNN
 F 2 "Capacitor_THT:C_Disc_D5.0mm_W2.5mm_P2.50mm" H 5188 2350 50  0001 C CNN
@@
 AR Path="/6003F027/6032BA93" Ref="R401"  Part="1"
 AR Path="/60043462/6032BA93" Ref="R501"  Part="1"
-F 0 "R501" V 3880 4200 50  0000 C CNN
+F 0 "R201" V 3880 4200 50  0000 C CNN
 F 1 "0" V 3800 4200 50  0000 C CNN
 F 2 "Resistor_THT:R_Axial_DIN0204_L3.6mm_D1.6mm_P1.90mm_Vertical" V 3730 4200 50  0001 C CNN
@@
 AR Path="/6003F027/60485F83" Ref="U401"  Part="1"
 AR Path="/60043462/60485F83" Ref="U501"  Part="1"
-F 0 "U501" H 3000 4700 50  0000 C CNN
+F 0 "U201" H 3000 4700 50  0000 C CNN
 F 1 "ACS723xLCTR-05AB" H 3250 4600 50  0000 C CNN
 F 2 "Package_SO:SOIC-8_3.9x4.9mm_P1.27mm" H 2850 3900 50  0001 L CIN
@@
 AR Path="/6003A868/60487676" Ref="C301"  Part="1"
 AR Path="/6003F027/60487676" Ref="C401"  Part="1"
-F 0 "C501" V 3100 3950 50  0000 C CNN
+F 0 "C201" V 3100 3950 50  0000 C CNN
 F 1 "100nF" V 3000 4000 50  0000 C CNN
 F 2 "Capacitor_THT:C_Disc_D5.0mm_W2.5mm_P2.50mm" H 2938 3650 50  0001 C CNN
@@
 	3650 5100 3650 3400
 $Comp
-L L6203:L6203 IC401
+L Edurov:L6203 IC401
 U 1 1 60738BFF
 P 4800 3100
@@
 AR Path="/6003A868/60738BFF" Ref="IC301"  Part="1"
 AR Path="/60043462/60738BFF" Ref="IC501"  Part="1"
-F 0 "IC501" H 4800 3681 50  0000 C CNN
+F 0 "IC201" H 4800 3681 50  0000 C CNN
 F 1 "L6203" H 4800 3590 50  0000 C CNN
 F 2 "SnapEDA Library:MULTIWATT-11" H 4800 3100 50  0001 L BNN
