File: pcb/EduRov-motherboard/eduRov_motherboard.kicad_pcb (KiCad board)
At the start: 4 copper layers, 167.7 x 124.6 mm, 67 parts, among them IC201 L6203, IC301 L6203, IC401 L6203, IC501 L6203, P101 Battery connector, P102 Ext press, P103 Ext press, P104 Ext press, P105 HeadLight, P106 HeadLight, Q101 IRL540NPBF, U201 ACS723xLCTR-05AB, U301 ACS723xLCTR-05AB, U401 ACS723xLCTR-05AB, U501 ACS723xLCTR-05AB

Commit message: Motherboard rev 0.7
Parts:
- moved P102 3.56 mm to (170.2, 115.2)
Connections:
- A101 pad 27: +5V -> Net-(A101-Pad27)
- A101 pad 30: Net-(A101-Pad30) -> +Bat
Routing:
- net +Bat: track 44.9 -> 56.5 mm
- net PressMonitor: track 92.7 -> 96.3 mm
Other:
- board text added: "+ -"
- board text added: "Revision by: Simen August Tinderholt 10.08.2021"
- board text added: "eduROV motherboard v0.7 www.edurov.no"
- board text removed: "Revision by: Simen August Tinderholt 03.07.2021"
- board text removed: "eduROV motherboard v0.6 www.edurov.no"
