File: pcb/EduRov-motherboard/eduRov_motherboard.sch (KiCad schematic (older format))
At the start: 52 parts, among them P101 Battery connector, P102 Ext press, P103 Ext press, P104 Ext press, P105 HeadLight, P106 HeadLight, Q101 IRL540NPBF, U1 Arduino header, U10 Nut, U11 Ferrules for motor cables, U12 Standoff, U13 Ferrules for motor cables, U14 Nut, U15 Ferrules for motor cables, U16 Standoff, U17 Ferrules for motor cables, U18 Nut, U19 Ferrules for motor cables, U2 Arduino header, U20 Standoff, U21 Ferrules for motor cables, U22 Nut, U23 Ferrules for motor cables, U24 Standoff, U25 Micro SD Card, U3 Raspberry PI stacking header, U4 Temp sensor, U5 Pressure sensor, U6 Sense hat, U7 Camera, U8 Jumper wires, U9 Ferrules for motor cables

Commit message: Motherboard updates
Connections:
- net +3V3: no longer A101.17 (3V3)
Changed lines of the file:
@@
 	1    0    0    1
 $EndComp
-Text GLabel 6325 1725 1    60   Input ~ 0
-+3V3
 Wire Notes Line
 	475  5775 10700 5775

Commit message: Motherboard rev 0.7
Connections:
- net +5V: no longer A101.27 (+5V)
- net +Bat1: now also A101.30 (VIN)
Changed lines of the file:
@@
 Wire Wire Line
 	5175 2325 5725 2325
-Text GLabel 6425 1725 1    60   Input ~ 0
-+5V
 Text GLabel 12075 5875 0    60   Input ~ 0
 Sense4
@@
 	1    0    0    -1
 $EndComp
+Text GLabel 6125 1725 1    60   Input ~ 0
++Bat1
 $EndSCHEMATC
