File: pcb/EduRov_headlights/eduRov_headlights.kicad_pcb (KiCad board)
At the start: 2 copper layers, 25.5 x 23 mm, 18 parts, among them J101 Conn_01x01, J102 Conn_01x01

Commit message: Update PCBs after prototyping
Parts:
- removed J101, J102: Conn_01x01, Connector_Pin:Pin_D1.3mm_L11.0mm
- added V+101: Conn_01x02, TestPoint:TestPoint_THTPad_D1.5mm_Drill0.7mm, F.Cu at (140.9, 129.3)
- added V-101: Conn_01x02, TestPoint:TestPoint_THTPad_D1.5mm_Drill0.7mm, F.Cu at (138.4, 129.3)
- moved R104 105.9 mm to (133.2, 128.8), turned to 0 degrees
- moved R103 105.8 mm to (128.0, 128.8), turned to 0 degrees
- moved R102 105.6 mm to (122.9, 128.8), turned to 0 degrees
- moved R101 105.4 mm to (117.7, 128.8), turned to 0 degrees
- moved D112 85.3 mm to (139.1, 125.3)
- moved D111 85.2 mm to (139.1, 119.3)
- moved D109 85.2 mm to (132.5, 125.3)
- moved D110 85.2 mm to (139.1, 113.2)
- moved D108 85.2 mm to (132.5, 119.3)
- moved D106 85.1 mm to (126.0, 125.3)
- moved D107 85.1 mm to (132.5, 113.2)
- moved D105 85.1 mm to (126.0, 119.3)
- moved D103 85.1 mm to (119.4, 125.3)
- moved D104 85.0 mm to (126.0, 113.2)
- moved D102 85.0 mm to (119.4, 119.3)
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Connections:
- D101 pad 2: Net-(D101-Pad2) -> /V+
- D103 pad 1: /V- -> Net-(D103-Pad1)
- D104 pad 2: Net-(D104-Pad2) -> /V+
- D106 pad 1: /V- -> Net-(D106-Pad1)
- D107 pad 2: Net-(D107-Pad2) -> /V+
- D109 pad 1: /V- -> Net-(D109-Pad1)
- D110 pad 2: Net-(D110-Pad2) -> /V+
- D112 pad 1: /V- -> Net-(D112-Pad1)
- R101 pad 1: /V+ -> Net-(D103-Pad1)
- R101 pad 2: Net-(D101-Pad2) -> /V-
- R102 pad 1: /V+ -> Net-(D106-Pad1)
- R102 pad 2: Net-(D104-Pad2) -> /V-
- R103 pad 1: /V+ -> Net-(D109-Pad1)
- R103 pad 2: Net-(D107-Pad2) -> /V-
- R104 pad 1: /V+ -> Net-(D112-Pad1)
- R104 pad 2: Net-(D110-Pad2) -> /V-
Routing:
- net /V+: track 17.0 -> 39.7 mm
- net /V-: track 5.35 -> 21.8 mm
- net Net-(D112-Pad1): track 0.00 -> 7.35 mm
- net Net-(D109-Pad1): track 0.00 -> 5.96 mm
- net Net-(D110-Pad2): track 5.41 -> 0.00 mm
- net Net-(D106-Pad1): track 0.00 -> 4.78 mm
- net Net-(D103-Pad1): track 0.00 -> 4.20 mm
- net Net-(D107-Pad2): track 3.83 -> 0.00 mm
- net Net-(D101-Pad2): track 3.58 -> 0.00 mm
- net Net-(D104-Pad2): track 2.99 -> 0.00 mm
- removed copper zone on F.Cu, net /V-
Other:
- board size 25.5 x 23 mm -> 26.1 x 21.8 mm
- board text added: "V+ V-"
- board text added: "V- V+"
- board text removed: "DIODES"
- board text removed: "RESISTORS"
- board text removed: "V+"
- board text removed: "V-"

Commit message: Update headlights with better spacing and holes.
Parts:
- V+101: footprint TestPoint:TestPoint_THTPad_D1.5mm_Drill0.7mm -> TestPoint:TestPoint_THTPad_D2.5mm_Drill1.2mm
- V-101: footprint TestPoint:TestPoint_THTPad_D1.5mm_Drill0.7mm -> TestPoint:TestPoint_THTPad_D3.0mm_Drill1.5mm
- moved V-101 20.3 mm to (118.1, 130.0)
- moved R101 4.13 mm to (121.8, 128.0), turned to 270 degrees
- moved R102 3.65 mm to (126.5, 128.3), turned to 270 degrees
- moved R103 3.47 mm to (131.4, 128.3), turned to 270 degrees
- moved R104 3.15 mm to (136.3, 128.3), turned to 270 degrees
- moved V+101 1.03 mm to (140.7, 130.3)
Routing:
- net Net-(D112-Pad1): track 7.35 -> 4.14 mm
- net /V-: track 21.8 -> 18.7 mm
- net Net-(D109-Pad1): track 5.96 -> 3.43 mm
- net Net-(D106-Pad1): track 4.78 -> 3.19 mm
Other:
- board size 26.1 x 21.8 mm -> 26.1 x 23.2 mm
- board text added: "V+"
- board text added: "V-"
- board text added: "eduROV headlight v0.2"
- board text removed: "V+ V-"
- board text removed: "V- V+"
