File: pcb/EduRov_headlights/eduRov_headlights.sch (KiCad schematic (older format))
At the start: 18 parts, among them J101 Conn_01x01, J102 Conn_01x01

Commit message: Update PCBs after prototyping
Parts:
- removed J101, J102: Conn_01x01, Connector_Pin:Pin_D1.3mm_L11.0mm, symbol Connector_Generic:Conn_01x01
- added V+101, V-101: Conn_01x02, TestPoint:TestPoint_THTPad_D1.5mm_Drill0.7mm, symbol Connector_Generic:Conn_01x01
Connections:
- net V+: now also D101.2 (A), D104.2 (A), D107.2 (A), D110.2 (A), V+101.1 (Pin_1); no longer R101.1, R102.1, R103.1, R104.1
- net V-: now also R101.2, R102.2, R103.2, R104.2, V-101.1 (Pin_1); no longer D103.1 (K), D106.1 (K), D109.1 (K), D112.1 (K)
- new net: D103.1 (K), R101.1
- new net: D106.1 (K), R102.1
- new net: D109.1 (K), R103.1
- new net: D112.1 (K), R104.1
Other:
- note removed: "Designed for 12V supply.\nDiode fw voltage (V_fw) for our white leds is between 3.2V and 4.0V, \nwe'll use 3.6V for our calculations\nOperating current (I_led) for our white LEDs is roughly 20mA.\n\nWe then calculate the required resistance per LED chain as follows:\nR = V_r / I_r\nV_r = 12V - (V_fw * num_leds) = 12 - (3.6 * 3) = 1.2V\nR = 1.2V / 20mA = 60 Ohm\n\n60 Ohm is not a standard resistan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"

Commit message: Add rest of component descriptions.
Parts:
- D101, D102, D103, D104, D105, D106, D107, D108, D109, D110, D111, D112: Description (none) -> White LED 5mm diameter, 3.2Vf; Digikey reference (none) -> C512A-WNN-CZ0B0151-ND; Manufacturer (none) -> Cree Inc.; Part number (none) -> C512A-WNN-CZ0B0151
- R101, R102, R103, R104: Description (none) -> 56 Ohm, 1/4W, 5%; Digikey reference (none) -> CF14JT56R0CT-ND; Manufacturer (none) -> Stackpole Electronics Inc; Part number (none) -> CF14JT56R0
Changed lines of the file:
@@
 F 2 "LED_THT:LED_D5.0mm_Clear" H 3250 3150 50  0001 C CNN
 F 3 "~" H 3250 3150 50  0001 C CNN
+F 4 "White LED 5mm diameter, 3.2Vf" H 3250 3150 50  0001 C CNN "Description"
+F 5 "C512A-WNN-CZ0B0151-ND" H 3250 3150 50  0001 C CNN "Digikey reference"
+F 6 "Cree Inc." H 3250 3150 50  0001 C CNN "Manufacturer"
+F 7 "C512A-WNN-CZ0B0151" H 3250 3150 50  0001 C CNN "Part number"
 	1    3250 3150
 	0    -1   -1   0
@@
 F 2 "LED_THT:LED_D5.0mm_Clear" H 3250 3450 50  0001 C CNN
 F 3 "~" H 3250 3450 50  0001 C CNN
+F 4 "White LED 5mm diameter, 3.2Vf" H 3250 3450 50  0001 C CNN "Description"
+F 5 "C512A-WNN-CZ0B0151-ND" H 3250 3450 50  0001 C CNN "Digikey reference"
+F 6 "Cree Inc." H 3250 3450 50  0001 C CNN "Manufacturer"
+F 7 "C512A-WNN-CZ0B0151" H 3250 3450 50  0001 C CNN "Part number"
 	1    3250 3450
 	0    -1   -1   0
@@
 F 2 "LED_THT:LED_D5.0mm_Clear" H 3250 3750 50  0001 C CNN
 F 3 "~" H 3250 3750 50  0001 C CNN
+F 4 "White LED 5mm diameter, 3.2Vf" H 3250 3750 50  0001 C CNN "Description"
+F 5 "C512A-WNN-CZ0B0151-ND" H 3250 3750 50  0001 C CNN "Digikey reference"
+F 6 "Cree Inc." H 3250 3750 50  0001 C CNN "Manufacturer"
+F 7 "C512A-WNN-CZ0B0151" H 3250 3750 50  0001 C CNN "Part number"
 	1    3250 3750
 	0    -1   -1   0
@@
 F 2 "Resistor_THT:R_Axial_DIN0207_L6.3mm_D2.5mm_P2.54mm_Vertical" V 3180 4050 50  0001 C CNN
 F 3 "~" H 3250 4050 50  0001 C CNN
+F 4 "56 Ohm, 1/4W, 5%" H 3250 4050 50  0001 C CNN "Description"
+F 5 "CF14JT56R0CT-ND" H 3250 4050 50  0001 C CNN "Digikey reference"
+F 6 "Stackpole Electronics Inc" H 3250 4050 50  0001 C CNN "Manufacturer"
+F 7 "CF14JT56R0" H 3250 4050 50  0001 C CNN "Part number"
 	1    3250 4050
 	1    0    0    -1
@@
 F 2 "LED_THT:LED_D5.0mm_Clear" H 3750 3150 50  0001 C CNN
 F 3 "~" H 3750 3150 50  0001 C CNN
+F 4 "White LED 5mm diameter, 3.2Vf" H 3750 3150 50  0001 C CNN "Description"
+F 5 "C512A-WNN-CZ0B0151-ND" H 3750 3150 50  0001 C CNN "Digikey reference"
+F 6 "Cree Inc." H 3750 3150 50  0001 C CNN "Manufacturer"
+F 7 "C512A-WNN-CZ0B0151" H 3750 3150 50  0001 C CNN "Part number"
 	1    3750 3150
 	0    -1   -1   0
@@
 F 2 "LED_THT:LED_D5.0mm_Clear" H 3750 3450 50  0001 C CNN
 F 3 "~" H 3750 3450 50  0001 C CNN
+F 4 "White LED 5mm diameter, 3.2Vf" H 3750 3450 50  0001 C CNN "Description"
+F 5 "C512A-WNN-CZ0B0151-ND" H 3750 3450 50  0001 C CNN "Digikey reference"
+F 6 "Cree Inc." H 3750 3450 50  0001 C CNN "Manufacturer"
+F 7 "C512A-WNN-CZ0B0151" H 3750 3450 50  0001 C CNN "Part number"
 	1    3750 3450
 	0    -1   -1   0
@@
 F 2 "LED_THT:LED_D5.0mm_Clear" H 3750 3750 50  0001 C CNN
 F 3 "~" H 3750 3750 50  0001 C CNN
+F 4 "White LED 5mm diameter, 3.2Vf" H 3750 3750 50  0001 C CNN "Description"
+F 5 "C512A-WNN-CZ0B0151-ND" H 3750 3750 50  0001 C CNN "Digikey reference"
+F 6 "Cree Inc." H 3750 3750 50  0001 C CNN "Manufacturer"
+F 7 "C512A-WNN-CZ0B0151" H 3750 3750 50  0001 C CNN "Part number"
 	1    3750 3750
 	0    -1   -1   0
@@
 F 2 "Resistor_THT:R_Axial_DIN0207_L6.3mm_D2.5mm_P2.54mm_Vertical" V 3680 4050 50  0001 C CNN
 F 3 "~" H 3750 4050 50  0001 C CNN
+F 4 "56 Ohm, 1/4W, 5%" H 3750 4050 50  0001 C CNN "Description"
+F 5 "CF14JT56R0CT-ND" H 3750 4050 50  0001 C CNN "Digikey reference"
+F 6 "Stackpole Electronics Inc" H 3750 4050 50  0001 C CNN "Manufacturer"
+F 7 "CF14JT56R0" H 3750 4050 50  0001 C CNN "Part number"
 	1    3750 4050
 	1    0    0    -1
@@
 F 2 "LED_THT:LED_D5.0mm_Clear" H 4250 3150 50  0001 C CNN
 F 3 "~" H 4250 3150 50  0001 C CNN
+F 4 "White LED 5mm diameter, 3.2Vf" H 4250 3150 50  0001 C CNN "Description"
+F 5 "C512A-WNN-CZ0B0151-ND" H 4250 3150 50  0001 C CNN "Digikey reference"
+F 6 "Cree Inc." H 4250 3150 50  0001 C CNN "Manufacturer"
+F 7 "C512A-WNN-CZ0B0151" H 4250 3150 50  0001 C CNN "Part number"
 	1    4250 3150
 	0    -1   -1   0
@@
 F 2 "LED_THT:LED_D5.0mm_Clear" H 4250 3450 50  0001 C CNN
 F 3 "~" H 4250 3450 50  0001 C CNN
+F 4 "White LED 5mm diameter, 3.2Vf" H 4250 3450 50  0001 C CNN "Description"
+F 5 "C512A-WNN-CZ0B0151-ND" H 4250 3450 50  0001 C CNN "Digikey reference"
+F 6 "Cree Inc." H 4250 3450 50  0001 C CNN "Manufacturer"
+F 7 "C512A-WNN-CZ0B0151" H 4250 3450 50  0001 C CNN "Part number"
 	1    4250 3450
 	0    -1   -1   0
@@
 F 2 "LED_THT:LED_D5.0mm_Clear" H 4250 3750 50  0001 C CNN
 F 3 "~" H 4250 3750 50  0001 C CNN
+F 4 "White LED 5mm diameter, 3.2Vf" H 4250 3750 50  0001 C CNN "Description"
+F 5 "C512A-WNN-CZ0B0151-ND" H 4250 3750 50  0001 C CNN "Digikey reference"
+F 6 "Cree Inc." H 4250 3750 50  0001 C CNN "Manufacturer"
+F 7 "C512A-WNN-CZ0B0151" H 4250 3750 50  0001 C CNN "Part number"
 	1    4250 3750
 	0    -1   -1   0
@@
 F 2 "Resistor_THT:R_Axial_DIN0207_L6.3mm_D2.5mm_P2.54mm_Vertical" V 4180 4050 50  0001 C CNN
 F 3 "~" H 4250 4050 50  0001 C CNN
+F 4 "56 Ohm, 1/4W, 5%" H 4250 4050 50  0001 C CNN "Description"
+F 5 "CF14JT56R0CT-ND" H 4250 4050 50  0001 C CNN "Digikey reference"
+F 6 "Stackpole Electronics Inc" H 4250 4050 50  0001 C CNN "Manufacturer"
+F 7 "CF14JT56R0" H 4250 4050 50  0001 C CNN "Part number"
 	1    4250 4050
 	1    0    0    -1
@@
 F 2 "LED_THT:LED_D5.0mm_Clear" H 4750 3150 50  0001 C CNN
 F 3 "~" H 4750 3150 50  0001 C CNN
+F 4 "White LED 5mm diameter, 3.2Vf" H 4750 3150 50  0001 C CNN "Description"
+F 5 "C512A-WNN-CZ0B0151-ND" H 4750 3150 50  0001 C CNN "Digikey reference"
+F 6 "Cree Inc." H 4750 3150 50  0001 C CNN "Manufacturer"
+F 7 "C512A-WNN-CZ0B0151" H 4750 3150 50  0001 C CNN "Part number"
 	1    4750 3150
 	0    -1   -1   0
@@
 F 2 "LED_THT:LED_D5.0mm_Clear" H 4750 3450 50  0001 C CNN
 F 3 "~" H 4750 3450 50  0001 C CNN
+F 4 "White LED 5mm diameter, 3.2Vf" H 4750 3450 50  0001 C CNN "Description"
+F 5 "C512A-WNN-CZ0B0151-ND" H 4750 3450 50  0001 C CNN "Digikey reference"
+F 6 "Cree Inc." H 4750 3450 50  0001 C CNN "Manufacturer"
+F 7 "C512A-WNN-CZ0B0151" H 4750 3450 50  0001 C CNN "Part number"
 	1    4750 3450
 	0    -1   -1   0
@@
 F 2 "LED_THT:LED_D5.0mm_Clear" H 4750 3750 50  0001 C CNN
 F 3 "~" H 4750 3750 50  0001 C CNN
+F 4 "White LED 5mm diameter, 3.2Vf" H 4750 3750 50  0001 C CNN "Description"
+F 5 "C512A-WNN-CZ0B0151-ND" H 4750 3750 50  0001 C CNN "Digikey reference"
+F 6 "Cree Inc." H 4750 3750 50  0001 C CNN "Manufacturer"
+F 7 "C512A-WNN-CZ0B0151" H 4750 3750 50  0001 C CNN "Part number"
 	1    4750 3750
 	0    -1   -1   0
@@
 F 2 "Resistor_THT:R_Axial_DIN0207_L6.3mm_D2.5mm_P2.54mm_Vertical" V 4680 4050 50  0001 C CNN
 F 3 "~" H 4750 4050 50  0001 C CNN
+F 4 "56 Ohm, 1/4W, 5%" H 4750 4050 50  0001 C CNN "Description"
+F 5 "CF14JT56R0CT-ND" H 4750 4050 50  0001 C CNN "Digikey reference"
+F 6 "Stackpole Electronics Inc" H 4750 4050 50  0001 C CNN "Manufacturer"
+F 7 "CF14JT56R0" H 4750 4050 50  0001 C CNN "Part number"
 	1    4750 4050
 	1    0    0    -1

Commit message: Generate boms using KiBom
Parts:
- V+101, V-101: Config (none) -> Do not place
Changed lines of the file:
@@
 F 2 "TestPoint:TestPoint_THTPad_D1.5mm_Drill0.7mm" H 2800 4200 50  0001 C CNN
 F 3 "~" H 2800 4200 50  0001 C CNN
+F 4 "Do not place" H 2800 4200 50  0001 C CNN "Config"
 	1    2800 4200
 	-1   0    0    1
@@
 F 2 "TestPoint:TestPoint_THTPad_D1.5mm_Drill0.7mm" H 2800 3000 50  0001 C CNN
 F 3 "~" H 2800 3000 50  0001 C CNN
+F 4 "Do not place" H 2800 3000 50  0001 C CNN "Config"
 	1    2800 3000
 	-1   0    0    1

Commit message: Update headlights with better spacing and holes.
Parts:
- V+101, V-101: footprint TestPoint:TestPoint_THTPad_D1.5mm_Drill0.7mm -> TestPoint:TestPoint_THTPad_D3.0mm_Drill1.5mm
Changed lines of the file:
@@
 F 0 "V-101" H 2800 4100 50  0000 C CNN
 F 1 "Conn_01x02" H 2800 4300 50  0000 C CNN
-F 2 "TestPoint:TestPoint_THTPad_D1.5mm_Drill0.7mm" H 2800 4200 50  0001 C CNN
+F 2 "TestPoint:TestPoint_THTPad_D3.0mm_Drill1.5mm" H 2800 4200 50  0001 C CNN
 F 3 "~" H 2800 4200 50  0001 C CNN
 F 4 "Do not place" H 2800 4200 50  0001 C CNN "Config"
@@
 F 0 "V+101" H 2800 2900 50  0000 C CNN
 F 1 "Conn_01x02" H 2800 3125 50  0000 C CNN
-F 2 "TestPoint:TestPoint_THTPad_D1.5mm_Drill0.7mm" H 2800 3000 50  0001 C CNN
+F 2 "TestPoint:TestPoint_THTPad_D3.0mm_Drill1.5mm" H 2800 3000 50  0001 C CNN
 F 3 "~" H 2800 3000 50  0001 C CNN
 F 4 "Do not place" H 2800 3000 50  0001 C CNN "Config"
